Commit message: fixed wheels model and arm joints,not fixed gazebo_ros_control errors

File: youbot_description/urdf/youbot.urdf.xacro (robot description, xacro)
@@ -75,10 +75,12 @@
       <visual>
         <geometry>
-          <sphere radius="${wheel_radius}"/>
+          <mesh filename="package://youbot_description/meshes/${position}_wheel.dae"/>
+          <!--sphere radius="${wheel_radius}"/-->
         </geometry>
       </visual>
       <collision>
         <geometry>
-          <sphere radius="${wheel_radius}"/>
+          <mesh filename="package://youbot_description/meshes/${position}_wheel.dae"/>
+          <!--sphere radius="${wheel_radius}"/-->
         </geometry>
       </collision>
@@ -140,5 +142,5 @@
     <!-- ### arm_2 ### -->
     <!-- arm_2 link -->
-    <!-- link name="arm_2_link">
+    <link name="arm_2_link">
       <inertial>
         <xacro:arm_2_inertial/>
@@ -149,7 +151,7 @@
         </geometry>
       </visual>
-    </link -->
+    </link >
     <!-- arm_2 joint -->
-    <!-- joint name="arm_2_joint" type="revolute">
+    <joint name="arm_2_joint" type="revolute">
       <xacro:arm_2_joint/>
       <child link="arm_2_link"/>
@@ -162,8 +164,8 @@
         <mechanicalReduction>1</mechanicalReduction>
       </actuator>
-    </transmission -->
+    </transmission >
     <!-- ### arm_3 ### -->
     <!-- arm_3 link -->
-    <!-- link name="arm_3_link">
+    <link name="arm_3_link">
       <inertial>
         <xacro:arm_3_inertial/>
@@ -174,7 +176,7 @@
         </geometry>
       </visual>
-    </link -->
+    </link >
     <!-- arm_3 joint -->
-    <!-- joint name="arm_3_joint" type="revolute">
+    <joint name="arm_3_joint" type="revolute">
       <xacro:arm_3_joint/>
       <child link="arm_3_link"/>
@@ -187,8 +189,8 @@
         <mechanicalReduction>1</mechanicalReduction>
       </actuator>
-    </transmission -->
+    </transmission >
     <!-- ### arm_4 ### -->
     <!-- arm_4 link -->
-    <!-- link name="arm_4_link">
+    <link name="arm_4_link">
       <inertial>
         <xacro:arm_4_inertial/>
@@ -199,7 +201,7 @@
         </geometry>
       </visual>
-    </link -->
+    </link >
     <!-- arm_4 joint -->
-    <!-- joint name="arm_4_joint" type="revolute">
+    <joint name="arm_4_joint" type="revolute">
       <xacro:arm_4_joint/>
       <child link="arm_4_link"/>
@@ -212,8 +214,8 @@
         <mechanicalReduction>1</mechanicalReduction>
       </actuator>
-    </transmission -->
+    </transmission>
     <!-- ### arm_5 ### -->
     <!-- arm_5 link -->
-    <!-- link name="arm_5_link">
+    <link name="arm_5_link">
       <inertial>
         <xacro:arm_5_inertial/>
@@ -224,7 +226,7 @@
         </geometry>
       </visual>
-    </link -->
+    </link >
     <!-- arm_5 joint -->
-    <!-- joint name="arm_5_joint" type="revolute">
+    <joint name="arm_5_joint" type="revolute">
       <xacro:arm_5_joint/>
       <child link="arm_5_link"/>
@@ -237,5 +239,5 @@
         <mechanicalReduction>1</mechanicalReduction>
       </actuator>
-    </transmission -->
+    </transmission >
   </xacro:macro>
   <xacro:macro name="gripper">
@@ -324,10 +326,10 @@
   </xacro:macro>
   <xacro:base/>
-  <xacro:wheels position="fl" x="1" y="-1"/>
-  <xacro:wheels position="fr" x="1" y="1"/>
-  <xacro:wheels position="bl" x="-1" y="-1"/>
-  <xacro:wheels position="br" x="-1" y="1"/>
+  <xacro:wheels position="front-left" x="1" y="-1"/>
+  <xacro:wheels position="front-right" x="1" y="1"/>
+  <xacro:wheels position="back-left" x="-1" y="-1"/>
+  <xacro:wheels position="back-right" x="-1" y="1"/>
   <xacro:arm_base/>
   <xacro:arm/>
-  <!-- xacro:gripper/ -->
+  <xacro:gripper/>
 </robot>
